File: hardware/osd.kicad_sch (KiCad schematic)
At the start: 21 parts, among them U10 SN74LVC1G3157DTBR, U11 COS8051SOT, U12 TLV7031DPWR

Commit message: Rev 2: finalize schematic + PCB for fabrication
Rev 2 change list implemented; on-canvas design annotations added across all
sheets (root, rp2350a, power, imu, osd, blackbox, pads). Design frozen for ordering.

Co-Authored-By: Claude Opus 4.8 (1M context) <noreply@anthropic.com>
Other:
- note added: "06/06/2026"
- note added: "2"
- note added: "75R input terminatiom"
- note added: "Analog OSD using PIO State Machine on RP2350"
- note added: "Analog switch (SPDT)"
- note added: "Comparator detects sync pulses, read by RP2350 PIO"
- note added: "Resistor divider let's GPIO port select between high (VOH = 1V: white) or low (VOL = 0.3v: black)"
- note removed: "Analog switch"

Commit message: chore(bom): consolidate LCSC Part -> LCSC field across schematic, library, footprints, project
Single canonical LCSC field (was split LCSC / LCSC Part). Every part resolves to one LCSC code; netlist verified, no duplicates. Includes Rev2 re-annotation resync re-save.

Co-Authored-By: Claude Opus 4.8 (1M context) <noreply@anthropic.com>
Parts:
- D8: LCSC (none) -> C151629; LCSC Part C151629 -> (none)
- U10: LCSC (none) -> C2673087; LCSC Part C2673087 -> (none)
- U11: LCSC (none) -> C7463385; LCSC Part C7463385 -> (none)
- U12: LCSC (none) -> C2876045; LCSC Part C2876045 -> (none)
Changed lines of the file:
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@@
 			)
 		)
-		(property "LCSC Part" "C2673087"
+		(property "LCSC" "C2673087"
 			(at 186.69 162.56 0)
 			(hide yes)
@@
 			)
 		)
-		(property "LCSC Part" "C7463385"
+		(property "LCSC" "C7463385"
 			(at 228.6 177.8 0)
 			(hide yes)
@@
 			)
 		)
-		(property "LCSC Part" "C2876045"
+		(property "LCSC" "C2876045"
 			(at 247.65 113.03 0)
 			(hide yes)
@@
 			)
 		)
-		(property "LCSC Part" "C151629"
+		(property "LCSC" "C151629"
 			(at 193.04 99.06 0)
 			(hide yes)
