File: hardware/pads.kicad_sch (KiCad schematic)
At the start: 57 parts, among them J1 5V, J10 5V, J11 5V, J12 5V, J13 5V, J14 5V, J15 5V, J16 5V, J17 5V, J18 5V, J19 5V, J2 5V, J20 5V, J21 5V, J22 5V, J23 5V, J24 5V, J25 5V, J26 5V, J27 5V, J28 5V, J29 5V, J3 5V, J30 5V, J31 5V, J32 5V, J33 5V, J34 5V, J35 5V, J36 5V, J37 5V, J38 5V, J39 5V, J4 5V, J40 5V, J41 5V, J42 5V, J43 5V, J44 5V, J45 5V, J46 5V, J47 5V, J48 5V, J49 5V, J5 5V, J50 5V, J51 5V, J52 5V, J53 5V, J54 5V, J55 5V, J6 5V, J7 5V, J8 5V, J9 5V, P1 SM08B-SRSS-TB(LF)(SN), U8 SM06B-SRSS-TB(LF)(SN)

Commit message: Rev 2: finalize schematic + PCB for fabrication
Rev 2 change list implemented; on-canvas design annotations added across all
sheets (root, rp2350a, power, imu, osd, blackbox, pads). Design frozen for ordering.

Co-Authored-By: Claude Opus 4.8 (1M context) <noreply@anthropic.com>
Other:
- note added: "06/06/2026"
- note added: "2"
- note added: "All solder pads broken out on the 30x30 lite variant"
- note added: "Solder pads and JST connectors for I/O"

Commit message: chore(bom): consolidate LCSC Part -> LCSC field across schematic, library, footprints, project
Single canonical LCSC field (was split LCSC / LCSC Part). Every part resolves to one LCSC code; netlist verified, no duplicates. Includes Rev2 re-annotation resync re-save.

Co-Authored-By: Claude Opus 4.8 (1M context) <noreply@anthropic.com>
Parts:
- P1: LCSC (none) -> C160407; LCSC Part C160407 -> (none)
- U8: LCSC (none) -> C160405; LCSC Part C160405 -> (none)
Changed lines of the file:
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@@
 			)
 		)
-		(property "LCSC Part" "C160405"
+		(property "LCSC" "C160405"
 			(at 161.29 64.77 0)
 			(hide yes)
@@
 			)
 		)
-		(property "LCSC Part" "C160407"
+		(property "LCSC" "C160407"
 			(at 105.41 29.21 0)
 			(hide yes)
