File: hardware/power.kicad_sch (KiCad schematic)
At the start: 34 parts, among them U3 TI LMR51430YFDDCR, U4 TI LMR51430YFDDCR, U5 TPS2116DRLR, U6 NCV8187AMT180TAG, U7 LP5912-3.3DRVR

Commit message: rev2 update
Parts:
- removed D10: RB161QS-40_C28646385, lib:SOD-882_L1.0-W0.6-RD, symbol lib:RB161QS-40_C28646385
- added D11: RB161QS-40_C28646385, lib:SOD-882_L1.0-W0.6-RD, symbol lib:RB161QS-40_C28646385
Connections:
- net +5V: now also D11.1 (C)
- net +5V_USB: now also D11.2 (A)

Commit message: routing
Parts:
- renumbered C24 to C22, C25 to C23, C26 to C24, C27 to C25, C28 to C26, C29 to C27, C30 to C28, C31 to C29, C32 to C30, C33 to C31, C34 to C32, D3 to D2, D11 to D3, D8 to D6, R27 to R19, R28 to R20, R29 to R21, R30 to R22, R31 to R23, R32 to R24, R33 to R25, R50 to R26, R40 to R27, R36 to R28
