File: hardware/rp2350a.kicad_sch (KiCad schematic)
At the start: 50 parts, among them Q2 DMN1150UFB-7B, Q3 DMN1150UFB-7B, U1 TS2306A 240GF MSM 9_C2976675, U2 RP2354B_C39843328, X1 XTM25012000JT00351001

Commit message: wip
Parts:
- removed C21: 100n, Capacitor_SMD:C_0201_0603Metric, symbol Device:C
- removed R16: 30R, Resistor_SMD:R_0201_0603Metric, symbol Device:R
- removed R17, R18: 4.7k, Resistor_SMD:R_0201_0603Metric, symbol Device:R
- removed R20: 1k, Resistor_SMD:R_0201_0603Metric, symbol Device:R
- removed R22, R25: 2.2k, Resistor_SMD:R_0201_0603Metric, symbol Device:R
- removed R26: 200R, Resistor_SMD:R_0201_0603Metric, symbol Device:R
- added R10, R9: 5.1k, Resistor_SMD:R_0201_0603Metric, symbol Device:R
- added R51: 2.4k, Resistor_SMD:R_0201_0603Metric, symbol Device:R
- added R52, R53: 75R, Resistor_SMD:R_0201_0603Metric, symbol Device:R
- Q2, Q3: value DMN1150UFB-7B -> AP1606; LCSC Part C459538 -> C2849580; MPN DMN1150UFB-7B -> AP1606; Manufacturer Diodes Incorporated -> (none)
Connections:
- net +3.3V: now also R10.1, R9.1; no longer Q3.1 (G)
- net +5V: now also R51.1
- net BEEPER: now also Q2.1 (G), R23.2
- net GND: now also Q3.2 (S)
- net I2C0.SCL: now also R9.2
- net LED0: now also R53.2
- net LED_STRIP: now also Q3.3 (D), R51.2
- net LED_STRIP_L: now also Q3.1 (G); no longer Q3.2 (S)
- net at D2.2 (A): now also R52.1
- new net: R52.2, R53.1
Other:
- note added: "RP2350 1.1V DC-DC SMPS Follow datasheet guidance on component placement"
- note added: "decoupling caps, place close to IC, one is enough when 2 pins are next to each other"
- note removed: "1.1V SMPS by RP datasheet inductor polarity important"
- note removed: "RC lowpass filters on ADC and VREG like Pico datasheet"
- note removed: "RP2350 1.8V DC-DC SMPS Follow datasheet guidance on component placement"
- note removed: "decoupling caps, place close to IC"
- moved on the sheet: C1, C10, C11, C12, C13, C14, C15, C16, C17, C18, C19, C20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

Commit message: rev2 update
Parts:
- removed D2: LED_1_Blue, LED_SMD:LED_0402_1005Metric, symbol Device:LED
- removed Q2, Q3: AP1606, lib:DFN-3L_L1.0-W0.6-P0.65-BR, symbol lib:DMN1150UFB-7B
- removed R10, R9: 5.1k, Resistor_SMD:R_0201_0603Metric, symbol Device:R
- removed R23: 100k, Resistor_SMD:R_0201_0603Metric, symbol Device:R
- added C21: 100n, Capacitor_SMD:C_0201_0603Metric, symbol Device:C
- added D10: LED_1_Blue, LED_SMD:LED_0402_1005Metric, symbol Device:LED
- added Q5, Q6: AP1606, lib:DFN-3L_L1.0-W0.6-P0.65-BR, symbol lib:DMN1150UFB-7B
- added R17, R18: 4.7k, Resistor_SMD:R_0201_0603Metric, symbol Device:R
- added R24: 100k, Resistor_SMD:R_0201_0603Metric, symbol Device:R
Connections:
- net +3.3V: now also C21.1, R17.2, R18.2
- net BEEPER: now also Q5.1 (G), R24.2
- net BUZZER-: now also Q5.3 (D)
- net GND: now also C21.2, D10.1 (K), Q5.2 (S), Q6.2 (S), R24.1
- net I2C0.SCL: now also R17.1
- net I2C0.SDA: now also R18.1
- net LED0: now also R52.1; no longer R53.2
- net LED_STRIP: now also Q6.3 (D)
- net LED_STRIP_L: now also Q6.1 (G)
- new net: D10.2 (A), R53.2
Other:
- note added: "1.1V SMPS by RP datasheet inductor polarity important"
- note added: "RC lowpass filters on ADC and VREG like Pico datasheet"
- note added: "RP2350 1.8V DC-DC SMPS Follow datasheet guidance on component placement"
- note added: "decoupling caps, place close to IC"
- note removed: "RP2350 1.1V DC-DC SMPS Follow datasheet guidance on component placement"
- note removed: "decoupling caps, place close to IC, one is enough when 2 pins are next to each other"
- moved on the sheet: C1, C10, C11, C12, C13, C14, C15, C16, C17, C18, C19, C20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

Commit message: lite done
Parts:
- removed C21: 100n, Capacitor_SMD:C_0201_0603Metric, symbol Device:C
- removed R17, R18: 4.7k, Resistor_SMD:R_0201_0603Metric, symbol Device:R
- added R10, R9: 5.1k, Resistor_SMD:R_0201_0603Metric, symbol Device:R
Connections:
- net +3.3V: now also Q6.1 (G), R10.1, R9.1
- net GND: no longer Q6.2 (S)
- net I2C0.SCL: now also R9.2
- net I2C0.SDA: now also R10.2
- net LED_STRIP_L: now also Q6.2 (S); no longer Q6.1 (G)
Other:
- note added: "decoupling caps, place close to IC, one is enough for two adjacent pins"
- note removed: "RP2350 1.8V DC-DC SMPS Follow datasheet guidance on component placement"
- note removed: "decoupling caps, place close to IC"
- moved on the sheet: C1, C10, C11, C12, C13, C17, C19, C3, C37, C4, C5, C6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

Commit message: routing
Parts:
- added C41: 100n, Capacitor_SMD:C_0201_0603Metric, symbol Device:C
- renumbered C9 to C10, C17 to C14, C14 to C15, C15 to C16, C16 to C17, C19 to C18, C18 to C19, C37 to C2, C23 to C21, C4 to C3, C6 to C4, C3 to C5, C5 to C6, C10 to C8, C8 to C9, D10 to D1, Q5 to Q1, Q6 to Q2, R12 to R10, R13 to R11, R14 to R12, R9 to R13, R10 to R14, R52 to R15, R53 to R16, R24 to R17, R51 to R18, R11 to R9
Connections:
- net +3.3V: now also C41.1
- net GND: now also C41.2
