File: hardware/rp2350a.kicad_sch (KiCad schematic)
At the start: 48 parts, among them Q1 AP1606, Q2 AP1606, U1 TS2306A 240GF MSM 9_C2976675, U2 RP2354B_C39843328, X1 XTM25012000JT00351001

Commit message: Rev 2: finalize schematic + PCB for fabrication
Rev 2 change list implemented; on-canvas design annotations added across all
sheets (root, rp2350a, power, imu, osd, blackbox, pads). Design frozen for ordering.

Co-Authored-By: Claude Opus 4.8 (1M context) <noreply@anthropic.com>
Other:
- note added: "06/06/2026"
- note added: "2"
- note added: "RP2350 Pin mapping and universal peripherals"
- moved on the sheet: C3, C4, C8, D1, Q1, Q2, R1, R13, R14, R15, R16, R17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

Commit message: chore(bom): consolidate LCSC Part -> LCSC field across schematic, library, footprints, project
Single canonical LCSC field (was split LCSC / LCSC Part). Every part resolves to one LCSC code; netlist verified, no duplicates. Includes Rev2 re-annotation resync re-save.

Co-Authored-By: Claude Opus 4.8 (1M context) <noreply@anthropic.com>
Parts:
- L1: LCSC (none) -> C42411119; LCSC Part C42411119 -> (none)
- Q1, Q2: LCSC (none) -> C2849580; LCSC Part C2849580 -> (none)
- U1: LCSC (none) -> C2976675; LCSC Part C2976675 -> (none)
- U2: LCSC (none) -> C39843328; LCSC Part C39843328 -> (none)
- USB1: LCSC (none) -> C5187472; LCSC Part C5187472 -> (none)
- X1: LCSC (none) -> C37635340; LCSC Part C37635340 -> (none)
Changed lines of the file:
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@@
 			)
 		)
-		(property "LCSC Part" "C2849580"
+		(property "LCSC" "C2849580"
 			(at 425.45 241.3 0)
 			(hide yes)
@@
 			)
 		)
-		(property "LCSC Part" "C5187472"
+		(property "LCSC" "C5187472"
 			(at 80.01 250.19 0)
 			(hide yes)
@@
 			)
 		)
-		(property "LCSC Part" "C39843328"
+		(property "LCSC" "C39843328"
 			(at 274.32 269.24 0)
 			(hide yes)
@@
 			)
 		)
-		(property "LCSC Part" "C42411119"
+		(property "LCSC" "C42411119"
 			(at 233.68 265.43 0)
 			(hide yes)
@@
 			)
 		)
-		(property "LCSC Part" "C2976675"
+		(property "LCSC" "C2976675"
 			(at 223.52 246.38 0)
 			(hide yes)
@@
 			)
 		)
-		(property "LCSC Part" "C37635340"
+		(property "LCSC" "C37635340"
 			(at 110.49 241.3 0)
 			(hide yes)
@@
 			)
 		)
-		(property "LCSC Part" "C2849580"
+		(property "LCSC" "C2849580"
 			(at 398.78 283.21 0)
 			(hide yes)
