File: hardware/OpenFC.kicad_pcb (KiCad board)
At the start: 6 copper layers, 37.5 x 37.5 mm, 164 parts, among them J1 5V, J10 5V, J11 5V, J12 5V, J13 5V, J14 5V, J15 5V, J18 5V, J2 5V, J21 5V, J22 5V, J25 5V, J26 5V, J27 5V, J28 5V, J29 5V, J30 5V, J31 5V, J32 5V, J33 5V, J34 5V, J35 5V, J36 5V, J37 5V, J38 5V, J39 5V, J4 5V, J40 5V, J41 5V, J42 5V, J43 5V, J44 5V, J45 5V, J46 5V, J47 5V, J48 5V, J49 5V, J5 5V, J50 5V, J52 5V, J53 5V, J54 5V, J7 5V, J8 5V, P1 SM08B-SRSS-TB(LF)(SN), Q1 DMN1150UFB-7B, Q2 DMN1150UFB-7B, Q3 DMN1150UFB-7B, Q4 DMN1150UFB-7B, U1 TS2306A 240GF MSM 9_C2976675, U18 SN74LVC1G3157DTBR, U19 TLV9061IDPWR, U2 RP2354B_C39843328, U20 TLV3201AIDBVR, U3 LMR51420YFDDCR, U4 LMR51420YFDDCR, U5 TPS2116DRLR, U6 NCV8187AMT180TAG, U7 LP5912-3.3DRVR, U8 SM06B-SRSS-TB(LF)(SN), U9 LSM6DSV16XTR, X1 XTM25012000JT00351001

Commit message: rev2 update
Parts:
- removed C2, C22, C43: 100n, Capacitor_SMD:C_0201_0603Metric
- removed Card1: TF-021B-H265, lib:TF-SMD_TF-021B-H265
- removed D1: USBLC6-2P6, Package_TO_SOT_SMD:SOT-666
- removed D2: LED_1_Green, LED_SMD:LED_0201_0603Metric
- removed D6: RB161QS-40_C28646385, lib:SOD-882_L1.0-W0.6-RD
- removed J53: 5V, lib:small_pad
- removed Q1, Q2, Q3, Q4: DMN1150UFB-7B, lib:DFN-3L_L1.0-W0.6-P0.65-BR
- removed R10, R15, R35, R39: 10k, Resistor_SMD:R_0201_0603Metric
- removed R16: 30R, Resistor_SMD:R_0201_0603Metric
- removed R19, R20: 1k, Resistor_SMD:R_0201_0603Metric
- removed R21, R23: 100k, Resistor_SMD:R_0201_0603Metric
- removed R22, R25: 2.2k, Resistor_SMD:R_0201_0603Metric
- removed R26, R34, R9: 200R, Resistor_SMD:R_0201_0603Metric
- removed U19: TLV9061IDPWR, lib:X2SON-4_L0.8-W0.8-P0.48-TL-DPW
- removed U20: TLV3201AIDBVR, lib:SOT-23-5_L3.0-W1.7-P0.95-LS2.8-BR
- added C37: 4.7uF, Capacitor_SMD:C_0402_1005Metric, F.Cu at (119.7, 69.8)
- added C44: 100n, Capacitor_SMD:C_0201_0603Metric, B.Cu at (138.8, 118.7)
- added Card2: TF PUSH, lib:TF-SMD_TF-PUSH, B.Cu at (145.3, 87.3)
- added D11: RB161QS-40_C28646385, lib:SOD-882_L1.0-W0.6-RD, F.Cu at (112.8, 65.9)
- added D8: LED_1_Green, LED_SMD:LED_0402_1005Metric, F.Cu at (106.6, 79.0)
- added J16: 5V, lib:small_pad, F.Cu at (162.2, 99.7)
- added J17: 5V, lib:small_pad, F.Cu at (140.7, 96.2)
- added J19: 5V, lib:small_pad, F.Cu at (142.4, 97.9)
- added J20: 5V, lib:small_pad, F.Cu at (163.9, 98.0)
- added J23: 5V, lib:small_pad, F.Cu at (162.1, 74.7)
- added J24: 5V, lib:small_pad, F.Cu at (165.6, 96.3)
- added J3: 5V, lib:small_pad, F.Cu at (165.5, 78.1)
- added J55: 5V, lib:small_pad, F.Cu at (153.1, 103.5)
- added J6: 5V, lib:small_pad, F.Cu at (142.3, 76.4)
- added J9: 5V, lib:small_pad, F.Cu at (144.1, 99.6)
- added Q5: AP1606, lib:DFN-3L_L1.0-W0.6-P0.65-BR, F.Cu at (119.3, 64.2)
- added Q6: AP1606, lib:DFN-3L_L1.0-W0.6-P0.65-BR, F.Cu at (119.3, 66.0)
- added R49: 10k, Resistor_SMD:R_0201_0603Metric, F.Cu at (109.2, 85.5)
- added R50: 2.4k, Resistor_SMD:R_0201_0603Metric, F.Cu at (102.5, 69.4)
- added R51: 2.4k, Resistor_SMD:R_0201_0603Metric, F.Cu at (117.0, 72.9)
- added R52: 75R, Resistor_SMD:R_0201_0603Metric, F.Cu at (117.0, 74.7)
- added R53: 75R, Resistor_SMD:R_0201_0603Metric, F.Cu at (117.0, 76.4)
- added R54: 10k, Resistor_SMD:R_0201_0603Metric, B.Cu at (138.8, 120.4)
- added TP1: TestPoint, TestPoint:TestPoint_Pad_D1.5mm, F.Cu at (96.0, 87.3)
- added TP2: TestPoint, TestPoint:TestPoint_Pad_D1.5mm, F.Cu at (96.0, 90.8)
- added TP3: TestPoint, TestPoint:TestPoint_Pad_D1.5mm, F.Cu at (96.0, 94.4)
- added TP4: TestPoint, TestPoint:TestPoint_Pad_D1.5mm, F.Cu at (96.0, 97.9)
- added U10: COS8051SOT, lib:SOT-23-5_L3.0-W1.7-P0.95-LS2.8-BR, F.Cu at (123.3, 88.4)
- added U11: TLV7031DPWR, lib:X2SON-4_L0.8-W0.8-P0.48-TL-A, B.Cu at (156.4, 137.8)
- C14, C15, C16, C24, C25, C26, C27, C28, C29, C30, C31, C32, C33, C34, C38, C39, C40, C41, C42, D3, D9, J10, J4, J7, L2, L3, R27, R28, R29, R31, R32, R41, R42, R43, R44, R45, R48, U18, U5, U6, U7: moved to F.Cu
- C21: value 4.7uF -> 100n; footprint Capacitor_SMD:C_0402_1005Metric -> Capacitor_SMD:C_0201_0603Metric; moved to F.Cu
- D10: value LED_1_Green -> LED_1_Blue; footprint LED_SMD:LED_0201_0603Metric -> LED_SMD:LED_0402_1005Metric
- D4, D5, D7: footprint LED_SMD:LED_0201_0603Metric -> LED_SMD:LED_0402_1005Metric
- R17, R18: value 2.2k -> 4.7k
- R24: value 10k -> 100k; moved to F.Cu
- R30: value 6.8k -> 6.49k; moved to F.Cu
- R33: value 470R -> 7.5k; moved to F.Cu
- R36: value 30R -> 510R; moved to F.Cu
- R40: value 200R -> 2.4k; moved to F.Cu
- R46, R47: value 470R -> 510R; moved to F.Cu
- U3, U4: value LMR51420YFDDCR -> TI LMR51430YFDDCR; moved to F.Cu
- moved C26 71.3 mm to (97.6, 64.2), turned to 0 degrees
- moved R29 66.2 mm to (100.1, 65.9), turned to 0 degrees
- moved R30 65.8 mm to (100.1, 67.7), turned to 0 degrees
- moved C28 63.4 mm to (98.4, 78.0)
- moved C31 62.7 mm to (97.6, 67.7), turned to 0 degrees
- moved L2 61.5 mm to (98.5, 74.4), turned to 0 degrees
- moved U3 61.1 mm to (106.2, 65.5), turned to 0 degrees
- moved C33 57.4 mm to (101.9, 79.7), turned to 0 degrees
- moved R40 54.5 mm to (102.5, 67.7), turned to 0 degrees
- moved C32 52.1 mm to (97.6, 69.4), turned to 0 degrees
- moved U6 51.8 mm to (110.0, 65.0), turned to 0 degrees
- moved C27 51.7 mm to (97.6, 65.9), turned to 0 degrees
- moved C24 51.7 mm to (110.3, 73.6)
- moved R28 51.1 mm to (100.1, 64.2)
- moved R27 50.7 mm to (97.6, 71.2)
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Connections:
- net /I2C_SDA renamed /PADS/I2C0.SDA
- net /IMU/GYRO_CS renamed /IMU/CS
- net /IMU/SPI0.CLKIN renamed /IMU/CLKIN
- net /PADS/DIGITAL_RX renamed /PADS/UART0_RX
- net /PADS/DIGITAL_TX renamed /PADS/UART0_TX
- net /UART1_TX renamed /PADS/UART1_TX
- C14 pad 1: GND -> Net-(U2-GPIO40_ADC0)
- C14 pad 2: /PADS/CURRENT -> GND
- C15 pad 1: GND -> Net-(U2-GPIO45_ADC5)
- C15 pad 2: /PADS/RSSI -> GND
- C16 pad 1: GND -> Net-(U2-GPIO47_ADC7)
- C16 pad 2: /PADS/ADC2 -> GND
- C21 pad 1: Net-(U2-ADC_AVDD) -> +3.3V
- D10 pad 1: Net-(D10-K) -> GND
- D10 pad 2: +5V -> Net-(D10-A)
- J10 pad 1: /LED -> /PADS/LED_STRIP
- J15 pad 1: /I2C_SCL -> /PADS/I2C0.SCL
- J54 pad 1: /PADS/PIOUART1_RX -> /PADS/PU1RX
- J8 pad 1: /UART1_RX -> /PADS/U1RX
- P1 pad 4: unconnected-(P1-Pad4) -> /PADS/PU1RX
- R1 pad 1: +BATT -> /RP2350A/ADC_VBAT
- R1 pad 2: /RP2350A/ADC_VBAT -> +BATT
- R17 pad 1: +3.3V -> /PADS/I2C0.SCL
- R17 pad 2: /I2C_SCL -> +3.3V
- R24 pad 1: /RP2350A/SBUS_INVERT -> GND
- R24 pad 2: +3.3V -> /RP2350A/BEEPER
- R40 pad 1: Net-(D10-K) -> Net-(D8-K)
- R40 pad 2: Net-(Q4-D) -> /POWER/1.8V_PG
- R46 pad 1: GND -> Net-(U10-IN-)
- R46 pad 2: Net-(U19-IN-) -> GND
- R47 pad 1: Net-(U19-IN-) -> Net-(U10-IN-)
- U2 pad 17: /I2C_SCL -> /PADS/I2C0.SCL
- U2 pad 21: /UART1_RX -> /PADS/U1RX
- U2 pad 28: /PADS/PIOUART1_RX -> /PADS/PU1RX
- U2 pad 35: Net-(U2-RUN) -> +3.3V
- U2 pad 59: Net-(U2-ADC_AVDD) -> +3.3V
- U2 pad 7: /RP2350A/SBUS_INVERT -> unconnected-(U2-GPIO9-Pad7)
- U8 pad 6: /PADS/SBUS -> /PADS/U1RX
Routing:
- net GND: track 106.8 -> 0.00 mm, vias 61 -> 0
- net +3.3V: track 87.7 -> 0.00 mm, vias 31 -> 0
- net +BATT: track 70.5 -> 0.00 mm, vias 9 -> 0
- net +10V: track 56.2 -> 0.00 mm, vias 5 -> 0
- net +1.1V: track 31.0 -> 0.00 mm, vias 5 -> 0
- net +5V: track 29.9 -> 0.00 mm, vias 21 -> 0
- net /BLACKBOX/SPI1.MISO: track 21.6 -> 0.00 mm, vias 2 -> 0
- net /POWER/10V_ENABLE: track 19.9 -> 0.00 mm, vias 2 -> 0
- net /BLACKBOX/FLASH_CS: track 18.3 -> 0.00 mm, vias 2 -> 0
- net /BLACKBOX/SPI1.SCK: track 16.9 -> 0.00 mm, vias 2 -> 0
- net /RP2350A/LED0: track 16.3 -> 0.00 mm, vias 2 -> 0
- net Net-(D10-K): track 16.0 -> 0.00 mm, vias 2 -> 0
- net /BLACKBOX/SPI1.MOSI: track 15.9 -> 0.00 mm, vias 2 -> 0
- net /PADS/RSSI: track 15.6 -> 0.00 mm, vias 2 -> 0
- net +5V_BUCK: track 14.7 -> 0.00 mm, vias 2 -> 0
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- removed copper zone on In2.Cu, net GND
Other:
- board size 37.5 x 37.5 mm -> 38.9 x 38.9 mm
- board text removed: "SBUS"

Commit message: routing
Parts:
- removed the C19 at (115.5, 107.1)
- removed the C21 at (117.0, 69.4)
- removed the C3 at (118.0, 112.0)
- removed the C34 at (101.9, 81.6)
- removed C42, C44: 100n, Capacitor_SMD:C_0201_0603Metric
- removed the C9 at (120.5, 112.8)
- removed D10: LED_1_Blue, LED_SMD:LED_0402_1005Metric
- removed D9: SDM02U30LP3-7B, lib:X3-DFN0603-2_L0.6-W0.3-RD
- removed Q5, Q6: AP1606, lib:DFN-3L_L1.0-W0.6-P0.65-BR
- removed the R12 at (113.4, 117.7)
- removed the R24 at (117.0, 71.2)
- removed R41, R48, R52, R53: 75R, Resistor_SMD:R_0201_0603Metric
- removed R42: 3.9k, Resistor_SMD:R_0201_0603Metric
- removed R43: 12k, Resistor_SMD:R_0201_0603Metric
- removed R44: 1.4k, Resistor_SMD:R_0201_0603Metric
- removed R45: 680R, Resistor_SMD:R_0201_0603Metric
- removed R46, R47: 510R, Resistor_SMD:R_0201_0603Metric
- removed R50, R51: 2.4k, Resistor_SMD:R_0201_0603Metric
- removed R54: 10k, Resistor_SMD:R_0201_0603Metric
- removed U18: SN74LVC1G3157DTBR, lib:X2SON-6_L1.0-W0.8-BL
- added C18: 100n, Capacitor_SMD:C_0201_0603Metric, B.Cu at (155.7, 81.5)
- added C2: 4.7uF, Capacitor_SMD:C_0402_1005Metric, B.Cu at (152.2, 82.8)
- added C30: 100n, Capacitor_SMD:C_0201_0603Metric, B.Cu at (159.3, 79.0)
- added C35: 100n, Capacitor_SMD:C_0201_0603Metric, B.Cu at (152.2, 88.3)
- added C36: 470p, Capacitor_SMD:C_0201_0603Metric, B.Cu at (160.1, 93.1)
- added C4: 20p, Capacitor_SMD:C_0201_0603Metric, B.Cu at (155.9, 83.2)
- added C8: 20p, Capacitor_SMD:C_0201_0603Metric, B.Cu at (154.7, 82.3)
- added D1: LED_1_Blue, LED_SMD:LED_0402_1005Metric, F.Cu at (159.5, 91.3)
- added D8: SDM02U30LP3-7B, lib:X3-DFN0603-2_L0.6-W0.3-RD, B.Cu at (161.1, 95.3)
- added Q1: AP1606, lib:DFN-3L_L1.0-W0.6-P0.65-BR, F.Cu at (147.0, 84.7)
- added Q2: AP1606, lib:DFN-3L_L1.0-W0.6-P0.65-BR, B.Cu at (156.7, 82.5)
- added R10: 30R, Resistor_SMD:R_0201_0603Metric, F.Cu at (151.5, 93.3)
- added R14: 5.1k, Resistor_SMD:R_0201_0603Metric, B.Cu at (156.2, 86.2)
- added R15: 75R, Resistor_SMD:R_0201_0603Metric, B.Cu at (156.2, 87.0)
- added R16: 75R, Resistor_SMD:R_0201_0603Metric, F.Cu at (161.1, 91.3)
- added R25: 7.5k, Resistor_SMD:R_0201_0603Metric, F.Cu at (145.5, 102.2)
- added R26: 2.4k, Resistor_SMD:R_0201_0603Metric, F.Cu at (144.7, 71.7)
- added R28: 510R, Resistor_SMD:R_0201_0603Metric, F.Cu at (161.1, 93.5)
- added R30: 10k, Resistor_SMD:R_0201_0603Metric, B.Cu at (151.8, 87.2)
- added R31: 75R, Resistor_SMD:R_0201_0603Metric, B.Cu at (159.3, 93.1)
- added R32: 3.9k, Resistor_SMD:R_0201_0603Metric, B.Cu at (157.8, 96.6)
- added R34: 1.4k, Resistor_SMD:R_0201_0603Metric, B.Cu at (158.5, 96.6)
- added R35: 680R, Resistor_SMD:R_0201_0603Metric, B.Cu at (158.6, 93.1)
- added R37: 510R, Resistor_SMD:R_0201_0603Metric, B.Cu at (165.9, 93.8)
- added R38: 75R, Resistor_SMD:R_0201_0603Metric, B.Cu at (166.6, 93.8)
- added R9: 10k, Resistor_SMD:R_0201_0603Metric, F.Cu at (147.3, 95.4)
- added U12: TLV7031DPWR, lib:X2SON-4_L0.8-W0.8-P0.48-TL-A, B.Cu at (160.9, 96.6)
- C10: value 20p -> 100n
- C12, C5, R1, R2, R6, U9: moved to F.Cu
- C14, C16, C39, L2, L3, R36, TP1, TP2, TP3, TP4, U3, U4, U5, U7: moved to B.Cu
- C21: renamed from C23; moved to F.Cu
- C22: renamed from C24; moved to B.Cu
- C23: renamed from C25; moved to B.Cu
- C24: renamed from C26; moved to B.Cu
- C25: renamed from C27; moved to B.Cu
- C26: renamed from C28; moved to B.Cu
- C27: renamed from C29; moved to B.Cu
- C28: renamed from C30; moved to B.Cu
- C3: renamed from C4; moved to F.Cu
- C32: value 100n -> 22uF; footprint Capacitor_SMD:C_0201_0603Metric -> Capacitor_SMD:C_0402_1005Metric; moved to B.Cu
- C33: renamed from C35; moved to F.Cu
- C34: renamed from C36; moved to F.Cu
- C37: value 4.7uF -> 100n; footprint Capacitor_SMD:C_0402_1005Metric -> Capacitor_SMD:C_0201_0603Metric; moved to B.Cu
- C38: value 470p -> 1uF; footprint Capacitor_SMD:C_0201_0603Metric -> Capacitor_SMD:C_0402_1005Metric; moved to B.Cu
- C40: value 1uF -> 100n; footprint Capacitor_SMD:C_0402_1005Metric -> Capacitor_SMD:C_0201_0603Metric; moved to B.Cu
- C6: value 20p -> 100n; moved to F.Cu
- C9: renamed from C8; moved to F.Cu
- D2: renamed from D3; moved to B.Cu
- D3: renamed from D11; moved to B.Cu
- R11: value 10k -> 30R; moved to F.Cu
- R12: renamed from R14; moved to F.Cu
- R13: value 30R -> 5.1k
- R17: value 4.7k -> 100k; moved to F.Cu
- R18: value 4.7k -> 2.4k
- R19: renamed from R27; moved to B.Cu
- R20: renamed from R28; moved to B.Cu
- R21: renamed from R29; moved to B.Cu
- R22: renamed from R30; moved to B.Cu
- R23: renamed from R31; moved to B.Cu
- R24: renamed from R32; moved to B.Cu
- R29: renamed from R49; moved to B.Cu
- R33: value 7.5k -> 12k; moved to B.Cu
- U10: value COS8051SOT -> SN74LVC1G3157DTBR; footprint lib:SOT-23-5_L3.0-W1.7-P0.95-LS2.8-BR -> lib:X2SON-6_L1.0-W0.8-BL; moved to B.Cu
- U11: value TLV7031DPWR -> COS8051SOT; footprint lib:X2SON-4_L0.8-W0.8-P0.48-TL-A -> lib:SOT-23-5_L3.0-W1.7-P0.95-LS2.8-BR
- moved R36 68.5 mm to (165.1, 93.8), turned to 90 degrees
- moved TP4 68.1 mm to (164.1, 99.0), turned to 180 degrees
- moved R19 66.1 mm to (163.6, 75.3)
- moved TP2 65.7 mm to (161.6, 93.6), turned to 180 degrees
- moved TP3 65.4 mm to (161.2, 99.0), turned to 180 degrees
- moved R33 65.3 mm to (159.2, 96.6), turned to 90 degrees
- moved C29 64.2 mm to (159.2, 85.9)
- moved R20 63.1 mm to (162.2, 75.3), turned to 180 degrees
- moved R27 62.3 mm to (161.1, 89.0)
- moved C28 61.1 mm to (162.9, 78.7), turned to 180 degrees
- moved TP1 60.9 mm to (156.2, 96.7), turned to 180 degrees
- moved R3 60.2 mm to (161.9, 86.9), turned to 0 degrees
- moved R21 59.7 mm to (147.6, 102.1), turned to -90 degrees
- moved C31 59.2 mm to (160.8, 85.8), turned to 180 degrees
- moved C32 58.9 mm to (155.7, 79.0), turned to 90 degrees
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- renumbered C18 to C19, C31 to C29, C33 to C31, Card2 to Card1, D8 to D6, J9 to J10, J10 to J11, J13 to J12, J12 to J13, J49 to J48, J48 to J49, J46 to J51, J45 to J53, J11 to J8, J8 to J9, R40 to R27
Connections:
- C10 pad 1: GND -> +3.3V
- C10 pad 2: Net-(C10-Pad2) -> GND
- C14 pad 1: Net-(U2-GPIO40_ADC0) -> +3.3V
- C15 pad 1: Net-(U2-GPIO45_ADC5) -> Net-(U2-GPIO40_ADC0)
- C16 pad 1: Net-(U2-GPIO47_ADC7) -> Net-(U2-GPIO45_ADC5)
- C17 pad 1: +3.3V -> Net-(U2-GPIO47_ADC7)
- C32 pad 1: +5V -> +3.3V
- C37 pad 1: +1.1V -> +3.3V
- C38 pad 2: GND -> /OSD/VID_DC
- C40 pad 1: /OSD/VID_FILT -> +3.3V
- C40 pad 2: /OSD/VID_DC -> GND
- C5 pad 1: +3.3V -> +1.1V
- C6 pad 1: GND -> +3.3V
- C6 pad 2: /RP2350A/XIN -> GND
- R11 pad 1: Net-(R11-Pad1) -> Net-(U2-USB_DP)
- R11 pad 2: Net-(U2-QSPI_SS) -> /RP2350A/D+
- R13 pad 1: Net-(U2-USB_DP) -> +3.3V
- R13 pad 2: /RP2350A/D+ -> /PADS/I2C0.SCL
- R17 pad 1: /PADS/I2C0.SCL -> GND
- R17 pad 2: +3.3V -> /RP2350A/BEEPER
- R18 pad 1: /PADS/I2C0.SDA -> +5V
- R18 pad 2: +3.3V -> /PADS/LED_STRIP
- R29 pad 2: +3V3 -> +3.3V
- R33 pad 1: +10V -> /OSD/OSD_LVL
- R33 pad 2: Net-(D4-A) -> +3.3V
- R36 pad 1: +3.3V -> Net-(U11-IN-)
- R36 pad 2: Net-(D7-A) -> GND
- R5 pad 2: Net-(C10-Pad2) -> Net-(C8-Pad2)
- TP1 pad 1: /OSD/VID_FILT -> /OSD/OSD_LVL
- TP2 pad 1: /OSD/VID_DC -> /OSD/VID_FILT
- TP3 pad 1: Net-(U10-IN+) -> /OSD/VID_DC
- TP4 pad 1: /OSD/OSD_LVL -> Net-(U10-A)
- U1 pad 2: Net-(R11-Pad1) -> Net-(R9-Pad1)
- U10 pad 1: Net-(U10-OUT) -> /OSD/OSD_LVL
- U10 pad 3: Net-(U10-IN+) -> /OSD/VIDEO_IN
- U10 pad 4: Net-(U10-IN-) -> Net-(U10-A)
- U11 pad 1: /OSD/OSD_SYNC -> Net-(U11-OUT)
- U11 pad 2: +3.3V -> GND
- U11 pad 3: GND -> Net-(U10-A)
- U11 pad 4: /OSD/VID_DC -> Net-(U11-IN-)
- U11 pad 5: GND -> +3.3V
- X1 pad 3: Net-(C10-Pad2) -> Net-(C8-Pad2)
Routing:
- net /PADS/LED_STRIP: track 0.00 -> 104.4 mm, vias 0 -> 7
- net GND: track 0.00 -> 60.9 mm, vias 0 -> 450
- net +3.3V: track 0.00 -> 50.9 mm, vias 0 -> 22
- net +5V: track 0.00 -> 50.4 mm, vias 0 -> 26
- net +BATT: track 0.00 -> 45.7 mm, vias 0 -> 7
- net +10V: track 0.00 -> 42.9 mm, vias 0 -> 8
- net +1.1V: track 0.00 -> 38.1 mm, vias 0 -> 6
- net /PADS/U1RX: track 0.00 -> 37.9 mm, vias 0 -> 2
- net +5V_BUCK: track 0.00 -> 28.6 mm, vias 0 -> 1
- net /PADS/PU1RX: track 0.00 -> 28.6 mm, vias 0 -> 3
- net /PADS/RSSI: track 0.00 -> 19.4 mm, vias 0 -> 3
- net /PADS/PIOUART1_TX: track 0.00 -> 19.4 mm, vias 0 -> 2
- net /PADS/UART0_RX: track 0.00 -> 19.1 mm, vias 0 -> 3
- net /POWER/10V_ENABLE: track 0.00 -> 18.9 mm, vias 0 -> 2
- net /PADS/UART1_TX: track 0.00 -> 18.9 mm, vias 0 -> 1
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- added copper zone on In3.Cu, net +3.3V
Other:
- board text added: "+"
- board text added: "-"
- board text added: "1"
- board text added: "10V buck"
- board text added: "10v buck"
- board text added: "2"
- board text added: "3"
- board text added: "3v3 LDO"
- board text added: "4"
- board text added: "5v buck"
- board text added: "5v power switch"
- board text added: "C"
- board text added: "G"
- board text added: "Lite"
- board text added: "OSD PIO"
- board text added: "OSDLVL"
- board text added: "R0"
- board text added: "SPDT"
- board text added: "Status"
- board text added: "T"
- board text added: "T0"
- board text added: "T1"
- board text added: "VID_DC"
- board text added: "crystal"
- board text added: "gyro"
- board text removed: "+5v"
- board text removed: "ECO"
- board text removed: "gnd"
- board text removed: "led"

Commit message: wip
Parts:
- removed R30: 10k, Resistor_SMD:R_0201_0603Metric
- moved C7 2.04 mm to (154.9, 92.0)
- turned J52 to 0 degrees
- turned J54 to 0 degrees
Routing:
- net +3.3V: track 50.9 -> 49.1 mm, vias 22 -> 23
- net /IMU/CLKIN: track 6.40 -> 7.72 mm
- net GND: track 60.9 -> 62.1 mm, vias 450 -> 447
- net /PADS/M1: track 12.4 -> 12.9 mm
- net /PADS/PIOUART0_RX: vias 1 -> 2
- added copper zone on In3.Cu, net +1.1V
Other:
- board text added: "R1"
- board text removed: "T1"

Commit message: reinsert resistor that kicad randomly deleted
Parts:
- added R30: 10k, Resistor_SMD:R_0201_0603Metric, B.Cu at (151.9, 87.2)
Changed lines of the file:
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@@
 		(sheetname "/PADS/")
 		(sheetfile "pads.kicad_sch")
+		(units
+			(unit
+				(name "A")
+				(pins "1")
+			)
+		)
 		(attr smd exclude_from_bom)
 		(duplicate_pad_numbers_are_jumpers no)
@@
 		(sheetname "/PADS/")
 		(sheetfile "pads.kicad_sch")
+		(units
+			(unit
+				(name "A")
+				(pins "1")
+			)
+		)
 		(attr smd exclude_from_bom)
 		(duplicate_pad_numbers_are_jumpers no)
@@
 		(sheetname "/PADS/")
 		(sheetfile "pads.kicad_sch")
+		(units
+			(unit
+				(name "A")
+				(pins "1")
+			)
+		)
 		(attr smd exclude_from_bom)
 		(duplicate_pad_numbers_are_jumpers no)
@@
 		(sheetname "/BLACKBOX/")
 		(sheetfile "blackbox.kicad_sch")
+		(units
+			(unit
+				(name "A")
+				(pins "1" "2" "3" "4" "5" "6" "7" "8" "CD" "13" "10" "12" "11")
+			)
+		)
 		(attr smd)
 		(duplicate_pad_numbers_are_jumpers no)
@@
 		(sheetname "/OSD/")
 		(sheetfile "osd.kicad_sch")
+		(units
+			(unit
+				(name "A")
+				(pins "3" "1" "5" "2" "4" "6")
+			)
+		)
 		(attr smd)
 		(duplicate_pad_numbers_are_jumpers no)
@@
 			(pintype "passive")
 		)
+		(embedded_fonts no)
+		(model "${KICAD10_3DMODEL_DIR}/Resistor_SMD.3dshapes/R_0201_0603Metric.step"
+			(offset
+				(xyz 0 0 0)
+			)
+			(scale
+				(xyz 1 1 1)
+			)
+			(rotate
+				(xyz 0 0 0)
+			)
+		)
+	)
+	(footprint "Resistor_SMD:R_0201_0603Metric"
+		(layer "B.Cu")
+		(at 151.865 87.205 90)
+		(descr "Resistor SMD 0201 (0603 Metric), square (rectangular) end terminal, IPC-7351 nominal, (Body size source: https://www.vishay.com/docs/20052/crcw0201e3.pdf)")
+		(tags "resistor")
+		(property "Reference" "R30"
+			(at 0 1.05 90)
+			(layer "B.SilkS")
+			(hide yes)
+			(effects
+				(font
+					(size 1 1)
+					(thickness 0.15)
+				)
+				(justify mirror)
+			)
+		)
+		(property "Value" "10k"
+			(at 0 -1.05 90)
+			(layer "B.Fab")
+			(hide yes)
+			(effects
+				(font
+					(size 1 1)
+					(thickness 0.15)
+				)
+				(justify mirror)
+			)
+		)
+		(property "Datasheet" ""
+			(at 0 0 90)
+			(layer "B.Fab")
+			(hide yes)
+			(effects
+				(font
+					(size 1.27 1.27)
+				)
+				(justify mirror)
+			)
+		)
+		(property "Description" "Resistor"
+			(at 0 0 90)
+			(layer "B.Fab")
+			(hide yes)
+			(effects
+				(font
+					(size 1.27 1.27)
+				)
+				(justify mirror)
+			)
+		)
+		(property "KiLib_Generator" "SMD_2terminal_chip_molded"
+			(at 0 0 90)
+			(layer "B.SilkS")
+			(hide yes)
+			(effects
+				(font
+					(size 1 1)
+					(thickness 0.15)
+				)
+				(justify mirror)
+			)
+		)
+		(property "LCSC" "C106225"
+			(at 0 0 270)
+			(unlocked yes)
+			(layer "B.Fab")
+			(hide yes)
+			(effects
+				(font
+					(size 1 1)
+					(thickness 0.15)
+				)
+				(justify mirror)
+			)
+		)
+		(property "MPN" "RC0201FR-0710KL"
+			(at 0 0 270)
+			(unlocked yes)
+			(layer "B.Fab")
+			(hide yes)
+			(effects
+				(font
+					(size 1 1)
+					(thickness 0.15)
+				)
+				(justify mirror)
+			)
+		)
+		(property "Manufacturer" "YAGEO"
+			(at 0 0 270)
+			(unlocked yes)
+			(layer "B.Fab")
+			(hide yes)
+			(effects
+				(font
+					(size 1 1)
+					(thickness 0.15)
+				)
+				(justify mirror)
+			)
+		)
+		(property ki_fp_filters "R_*")
+		(sheetname "/BLACKBOX/")
+		(sheetfile "blackbox.kicad_sch")
+		(units
+			(unit
+				(name "A")
+				(pins "1" "2")
+			)
+		)
+		(attr smd)
+		(duplicate_pad_numbers_are_jumpers no)
+		(fp_rect
+			(start -0.7 0.35)
+			(end 0.7 -0.35)
+			(stroke
+				(width 0.05)
+				(type solid)
+			)
+			(fill no)
+			(layer "B.CrtYd")
+		)
+		(fp_rect
+			(start -0.3 0.15)
+			(end 0.3 -0.15)
+			(stroke
+				(width 0.1)
+				(type solid)
+			)
+			(fill no)
+			(layer "B.Fab")
+		)
+		(fp_text user "${REFERENCE}"
+			(at 0 0.68 90)
+			(layer "B.Fab")
+			(effects
+				(font
+					(size 0.25 0.25)
+					(thickness 0.04)
+				)
+				(justify mirror)
+			)
+		)
+		(pad "" smd roundrect
+			(at -0.345 0 90)
+			(size 0.318 0.36)
+			(layers "B.Paste")
+			(roundrect_rratio 0.25)
+		)
+		(pad "" smd roundrect
+			(at 0.345 0 90)
+			(size 0.318 0.36)
+			(layers "B.Paste")
+			(roundrect_rratio 0.25)
+		)
+		(pad "1" smd roundrect
+			(at -0.32 0 90)
+			(size 0.46 0.4)
+			(layers "B.Cu" "B.Mask")
+			(roundrect_rratio 0.25)
+			(net "+3.3V")
+			(pintype "passive")
+		)
+		(pad "2" smd roundrect
+			(at 0.32 0 90)
+			(size 0.46 0.4)
+			(layers "B.Cu" "B.Mask")
+			(roundrect_rratio 0.25)
+			(net "/BLACKBOX/FLASH_CS")
+			(pintype "passive")
+		)
