File: hardware/imu.kicad_sch (KiCad schematic)
At the start: 4 parts, among them U9 LSM6DSV16XTR

Commit message: Rev 2: finalize schematic + PCB for fabrication
Rev 2 change list implemented; on-canvas design annotations added across all
sheets (root, rp2350a, power, imu, osd, blackbox, pads). Design frozen for ordering.

Co-Authored-By: Claude Opus 4.8 (1M context) <noreply@anthropic.com>
Other:
- note added: "06/06/2026"
- note added: "2"
- note added: "IMU SPI wiring and local decoupling"
- note added: "Universal IMU wiring and LGA footprint (BMI270, LSM6, TDK..)"

Commit message: chore(bom): consolidate LCSC Part -> LCSC field across schematic, library, footprints, project
Single canonical LCSC field (was split LCSC / LCSC Part). Every part resolves to one LCSC code; netlist verified, no duplicates. Includes Rev2 re-annotation resync re-save.

Co-Authored-By: Claude Opus 4.8 (1M context) <noreply@anthropic.com>
Parts:
- U9: LCSC (none) -> C5267406; LCSC Part C5267406 -> (none)
Changed lines of the file:
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@@
 			)
 		)
-		(property "LCSC Part" "C5267406"
+		(property "LCSC" "C5267406"
 			(at 72.39 87.63 0)
 			(hide yes)
